File: cuisinart-oven.brd (EAGLE design)
At the start: 43 parts, among them CN1 CN1, CON1 CON1, IC3 P1014AP06, IC4 PC817, K1 V23148-A0003-B101-NO, K2 V23148-A0003-B101-NO, T1 TICP206, T2 BD705

Commit message: Complete schematic
Finally the circuit is complete.
Parts:
- removed R6: 4700 Ohm, SparkFun-Resistors:AXIAL-0.3
- added C18, C19, C4, C5: (no value), rcl:C025-024X044
- added C31: 0.1 uF, rcl:XC15B6
- added D1, D4, D7: 1N4004, diode:DO41-10
- added L3: DS10, inductors:DS10
- added R20: 180000 Ohm, SparkFun-Resistors:AXIAL-0.3
- added R30: 10000 Ohm, SparkFun-Resistors:AXIAL-0.3
- added R31, R33: 3300 Ohm, SparkFun-Resistors:AXIAL-0.3
- added R36: 4700 Ohm, SparkFun-Resistors:AXIAL-0.3
- added R45: 100 Ohm, SparkFun-Resistors:AXIAL-0.3
- added R46: 1000 Ohm, SparkFun-Resistors:AXIAL-0.3
- C3: value 0.1 uF -> (none); device rcl:XC15B6 -> rcl:C025-024X044
- R3: value 100 Ohm -> 3300 Ohm
- moved C3 414.0 mm to (86.4, -649.0)
- moved R3 252.5 mm to (91.4, -613.4)
- moved R5 19.0 mm to (91.4, -575.3)
- renumbered R7 to R32, T3 to Q3, T4 to Q4, T5 to Q1, T6 to Q5
Connections:
- removed net N$24: C7.+, T2.3
- new net N$10: CON1.3, R36.P$1
- new net N$26: Q3.B, R3.P$2, R36.P$2
- new net N$27: Q3.C, R4.P$2
- new net N$28: C3.1, Q3.E, R46.P$2, T1.G
- new net N$29: CON1.8, Q1.C
- new net N$30: C5.1, Q5.B, R32.P$2, R33.P$2
- new net N$31: C19.2, C7.+, CON1.6, D4.A, R20.P$1, T2.3
- new net N$33: C4.1, Q4.B, R31.P$2, R5.P$2
- new net N$34: CON1.2, R32.P$1
- new net N$37: CON1.1, R5.P$1
- net N$12: now also L3.1
- net N$13: now also C31.2; no longer C3.2
- net N$14: now also C18.2, C28.-, C3.2, C4.2, C5.2, C7.-, CN1.1, CON1.4, D1.C, D3.C, D7.C, Q1.E, Q4.E, Q5.E, R16.P$2, R3.P$1, R30.P$1, R31.P$1, R33.P$1, R46.P$1, SG1.+, ZD1.C, ZD2.C
- net N$15: now also C31.1; no longer C3.1
- net N$19: now also C18.1, D1.A, Q1.B, R1.P$2, R30.P$2; no longer C28.-, C7.-, CN1.1, CON1.4, D3.C, R16.P$2, SG1.+, ZD1.C
- net N$21: now also R45.P$1; no longer R3.P$1
- net N$22: now also R45.P$2; no longer R3.P$2
- net N$25: now also C19.1, D4.C, D7.A, R20.P$2
- net N$6: now also Q4.C
- net N$8: now also Q5.C
- net VCC_2: now also L3.2
